Commit message: Update myrobot.urdf

File: 02_URDF/myrobot.urdf (robot description, URDF)
Before this commit: robot myrobot, 1 links, 0 joints
Links:
- added link box; visual box size=0.08 0.08 0.08
- added link head; visual sphere radius=0.2
- added link left_base; visual box size=0.4 0.1 0.1
- added link left_leg; visual box size=0.6 0.1 0.2
- added link right_base; visual box size=0.4 0.1 0.1
- added link right_leg; visual box size=0.6 0.1 0.2
- link base_link: geometry visual cylinder length=0.6 radius=0.2
Joints:
- added joint base_to_left_leg: type fixed, parent base_link, child left_leg, origin xyz=0 0.22 0.25
- added joint base_to_right_leg: type fixed, parent base_link, child right_leg, origin xyz=0 -0.22 0.25
- added joint head_swivel: type fixed, parent base_link, child head, origin xyz=0 0 0.32
- added joint left_base_joint: type fixed, parent left_leg, child left_base, origin xyz=0 0 -0.6
- added joint right_base_joint: type fixed, parent right_leg, child right_base, origin xyz=0 0 -0.6
- added joint tobox: type fixed, parent head, child box, origin xyz=0.1814 0 0.1414
