Commit message: add justin urdf

File: 02_URDF/iai_kitchen.urdf.xacro (robot description, xacro)
@@ -26,5 +26,5 @@
     <link name="world"/>
     <joint name="world_room_joint" type="fixed">
-      <origin xyz="0.0 0.03 0 " rpy="0 0 0" />
+      <origin xyz="0.0 0.03 0 " rpy="0 0 ${pi/2}" />
       <parent link="world"/>
       <child link="room_link"/>
